File: circuit/lpcounter.sch (KiCad schematic (older format))
At the start: 17 parts, among them IC1 ATTINY85V-P, M1 SYN115, P1 CONN_01X08

Commit message: proper battery holder for CR2032
Parts:
- BT1: footprint Buzzers_Beepers:Buzzer_12x9.5RM7.6 -> Battery_Holders:Keystone_106_1x20mm-CoinCell
Changed lines of the file:
@@
 F 0 "BT1" H 6300 5300 50  0000 L CNN
 F 1 "3.7V" H 6300 5200 50  0000 L CNN
-F 2 "Buzzers_Beepers:Buzzer_12x9.5RM7.6" V 6200 5260 50  0001 C CNN
+F 2 "Battery_Holders:Keystone_106_1x20mm-CoinCell" V 6200 5260 50  0001 C CNN
 F 3 "" V 6200 5260 50  0000 C CNN
 	1    6200 5200

Commit message: updating PCB
Parts:
- M1: footprint Connectors_Molex:Molex_KK-6410-04_04x2.54mm_Straight -> Pin_Headers:Pin_Header_Straight_1x04_Pitch2.00mm
Changed lines of the file:
@@
 F 0 "M1" H 9800 3750 50  0000 C CNN
 F 1 "SYN115" V 9900 3500 50  0000 C CNN
-F 2 "Connectors_Molex:Molex_KK-6410-04_04x2.54mm_Straight" H 9800 3500 50  0001 C CNN
+F 2 "Pin_Headers:Pin_Header_Straight_1x04_Pitch2.00mm" H 9800 3500 50  0001 C CNN
 F 3 "" H 9800 3500 50  0000 C CNN
 	1    9800 3500

Commit message: fully routed
Parts:
- added P2: CONN_02X01, Buttons_Switches_SMD:SW_SPST_SKQG, symbol CONN_02X01
- added R6: 10k, Resistors_SMD:R_1206_HandSoldering, symbol R
- P1: footprint Connectors_Molex:Molex_KK-6410-08_08x2.54mm_Straight -> Connectors_Phoenix:PhoenixContact_MSTBVA-G_08x5.08mm_Vertical
Connections:
- wire segments 29 -> 31
Changed lines of the file:
@@
 F 0 "P1" H 1350 4050 50  0000 C CNN
 F 1 "CONN_01X08" V 1450 3600 50  0000 C CNN
-F 2 "Connectors_Molex:Molex_KK-6410-08_08x2.54mm_Straight" H 1350 3600 50  0001 C CNN
+F 2 "Connectors_Phoenix:PhoenixContact_MSTBVA-G_08x5.08mm_Vertical" H 1350 3600 50  0001 C CNN
 F 3 "" H 1350 3600 50  0000 C CNN
 	1    1350 3600
@@
 	1    0    0    -1
 $EndComp
+$Comp
+L CONN_02X01 P2
+U 1 1 5910624E
+P 4350 5250
+F 0 "P2" H 4350 5350 50  0000 C CNN
+F 1 "CONN_02X01" H 4350 5150 50  0000 C CNN
+F 2 "Buttons_Switches_SMD:SW_SPST_SKQG" H 4350 4050 50  0001 C CNN
+F 3 "" H 4350 4050 50  0000 C CNN
+	1    4350 5250
+	0    -1   -1   0
+$EndComp
+$Comp
+L R R6
+U 1 1 591067B7
+P 4350 4650
+F 0 "R6" V 4430 4650 50  0000 C CNN
+F 1 "10k" V 4350 4650 50  0000 C CNN
+F 2 "Resistors_SMD:R_1206_HandSoldering" V 4280 4650 50  0001 C CNN
+F 3 "" H 4350 4650 50  0000 C CNN
+	1    4350 4650
+	1    0    0    -1
+$EndComp
+$Comp
+L +3V3 #PWR024
+U 1 1 591067BD
+P 4350 4500
+F 0 "#PWR024" H 4350 4350 50  0001 C CNN
+F 1 "+3V3" H 4350 4640 50  0000 C CNN
+F 2 "" H 4350 4500 50  0000 C CNN
+F 3 "" H 4350 4500 50  0000 C CNN
+	1    4350 4500
+	1    0    0    -1
+$EndComp
+Wire Wire Line
+	4350 4800 4350 5000
+Wire Wire Line
+	4350 4950 4850 4950
+Connection ~ 4350 4950
+$Comp
+L GND #PWR025
+U 1 1 59106977
+P 4350 5500
+F 0 "#PWR025" H 4350 5250 50  0001 C CNN
+F 1 "GND" H 4350 5350 50  0000 C CNN
+F 2 "" H 4350 5500 50  0000 C CNN
+F 3 "" H 4350 5500 50  0000 C CNN
+	1    4350 5500
+	1    0    0    -1
+$EndComp
+Text Label 4450 4950 0    60   ~ 0
+RESETn
 $EndSCHEMATC

Commit message: correct footprint for SYN115, 4 screw holes, optimizing PCB drawing 18650 battery outiline
Parts:
- added P3, P4, P5, P6: Hole_3.5mm, Mounting_Holes:MountingHole_3.5mm, symbol CONN_01X01
- M1: footprint Pin_Headers:Pin_Header_Straight_1x04_Pitch2.00mm -> syn115:SYN115
Changed lines of the file:
@@
 F 0 "M1" H 9800 3750 50  0000 C CNN
 F 1 "SYN115" V 9900 3500 50  0000 C CNN
-F 2 "Pin_Headers:Pin_Header_Straight_1x04_Pitch2.00mm" H 9800 3500 50  0001 C CNN
+F 2 "syn115:SYN115" H 9800 3500 50  0001 C CNN
 F 3 "" H 9800 3500 50  0000 C CNN
 	1    9800 3500
@@
 Text Label 4450 4950 0    60   ~ 0
 RESETn
+$Comp
+L CONN_01X01 P5
+U 1 1 59119B55
+P 2250 4600
+F 0 "P5" H 2250 4700 50  0000 C CNN
+F 1 "Hole_3.5mm" V 2350 4600 50  0000 C CNN
+F 2 "Mounting_Holes:MountingHole_3.5mm" H 2250 4600 50  0001 C CNN
+F 3 "" H 2250 4600 50  0000 C CNN
+	1    2250 4600
+	0    -1   -1   0
+$EndComp
+$Comp
+L GND #PWR026
+U 1 1 59119C8B
+P 2250 4800
+F 0 "#PWR026" H 2250 4550 50  0001 C CNN
+F 1 "GND" H 2250 4650 50  0000 C CNN
+F 2 "" H 2250 4800 50  0000 C CNN
+F 3 "" H 2250 4800 50  0000 C CNN
+	1    2250 4800
+	1    0    0    -1
+$EndComp
+$Comp
+L CONN_01X01 P6
+U 1 1 59119D21
+P 2800 4600
+F 0 "P6" H 2800 4700 50  0000 C CNN
+F 1 "Hole_3.5mm" V 2900 4600 50  0000 C CNN
+F 2 "Mounting_Holes:MountingHole_3.5mm" H 2800 4600 50  0001 C CNN
+F 3 "" H 2800 4600 50  0000 C CNN
+	1    2800 4600
+	0    -1   -1   0
+$EndComp
+$Comp
+L GND #PWR027
+U 1 1 59119D27
+P 2800 4800
+F 0 "#PWR027" H 2800 4550 50  0001 C CNN
+F 1 "GND" H 2800 4650 50  0000 C CNN
+F 2 "" H 2800 4800 50  0000 C CNN
+F 3 "" H 2800 4800 50  0000 C CNN
+	1    2800 4800
+	1    0    0    -1
+$EndComp
+$Comp
+L CONN_01X01 P3
+U 1 1 59119EC3
+P 1150 4600
+F 0 "P3" H 1150 4700 50  0000 C CNN
+F 1 "Hole_3.5mm" V 1250 4600 50  0000 C CNN
+F 2 "Mounting_Holes:MountingHole_3.5mm" H 1150 4600 50  0001 C CNN
+F 3 "" H 1150 4600 50  0000 C CNN
+	1    1150 4600
+	0    -1   -1   0
+$EndComp
+$Comp
+L GND #PWR028
+U 1 1 59119EC9
+P 1150 4800
+F 0 "#PWR028" H 1150 4550 50  0001 C CNN
+F 1 "GND" H 1150 4650 50  0000 C CNN
+F 2 "" H 1150 4800 50  0000 C CNN
+F 3 "" H 1150 4800 50  0000 C CNN
+	1    1150 4800
+	1    0    0    -1
+$EndComp
+$Comp
+L CONN_01X01 P4
+U 1 1 59119ECF
+P 1700 4600
+F 0 "P4" H 1700 4700 50  0000 C CNN
+F 1 "Hole_3.5mm" V 1800 4600 50  0000 C CNN
+F 2 "Mounting_Holes:MountingHole_3.5mm" H 1700 4600 50  0001 C CNN
+F 3 "" H 1700 4600 50  0000 C CNN
+	1    1700 4600
+	0    -1   -1   0
+$EndComp
+$Comp
+L GND #PWR029
+U 1 1 59119ED5
+P 1700 4800
+F 0 "#PWR029" H 1700 4550 50  0001 C CNN
+F 1 "GND" H 1700 4650 50  0000 C CNN
+F 2 "" H 1700 4800 50  0000 C CNN
+F 3 "" H 1700 4800 50  0000 C CNN
+	1    1700 4800
+	1    0    0    -1
+$EndComp
 $EndSCHEMATC

Commit message: 3V battery connected direct, 3.7V battery connect in series with diode 1N4147
Parts:
- added P7: BAT+, Pin_Headers:Pin_Header_Straight_1x01, symbol CONN_01X01
- added P8: BAT-, Pin_Headers:Pin_Header_Straight_1x01, symbol CONN_01X01
- BT1: value 3.7V -> CR2032
Other:
- moved on the sheet: D1
Changed lines of the file:
@@
 IN0
 $Comp
-L GND #PWR01
+L GND #PWR28
 U 1 1 591028B9
 P 7900 3850
-F 0 "#PWR01" H 7900 3600 50  0001 C CNN
+F 0 "#PWR28" H 7900 3600 50  0001 C CNN
 F 1 "GND" H 7900 3700 50  0000 C CNN
 F 2 "" H 7900 3850 50  0000 C CNN
@@
 RESETn
 $Comp
-L +3V3 #PWR02
+L +3V3 #PWR27
 U 1 1 59102AB8
 P 7900 3250
-F 0 "#PWR02" H 7900 3100 50  0001 C CNN
+F 0 "#PWR27" H 7900 3100 50  0001 C CNN
 F 1 "+3V3" H 7900 3390 50  0000 C CNN
 F 2 "" H 7900 3250 50  0000 C CNN
@@
 L D_ALT D1
 U 1 1 59102ADE
-P 6200 4850
-F 0 "D1" H 6200 4950 50  0000 C CNN
-F 1 "1N4148" H 6200 4750 50  0000 C CNN
-F 2 "Diodes_SMD:MELF_Handsoldering" H 6200 4850 50  0001 C CNN
-F 3 "" H 6200 4850 50  0000 C CNN
-	1    6200 4850
+P 5550 4950
+F 0 "D1" H 5550 5050 50  0000 C CNN
+F 1 "1N4148" H 5550 4850 50  0000 C CNN
+F 2 "Diodes_SMD:MELF_Handsoldering" H 5550 4950 50  0001 C CNN
+F 3 "" H 5550 4950 50  0000 C CNN
+	1    5550 4950
 	0    1    1    0
 $EndComp
 $Comp
-L +3V3 #PWR03
+L +3V3 #PWR21
 U 1 1 59102B87
-P 6200 4700
-F 0 "#PWR03" H 6200 4550 50  0001 C CNN
-F 1 "+3V3" H 6200 4840 50  0000 C CNN
-F 2 "" H 6200 4700 50  0000 C CNN
-F 3 "" H 6200 4700 50  0000 C CNN
-	1    6200 4700
+P 6200 5000
+F 0 "#PWR21" H 6200 4850 50  0001 C CNN
+F 1 "+3V3" H 6200 5140 50  0000 C CNN
+F 2 "" H 6200 5000 50  0000 C CNN
+F 3 "" H 6200 5000 50  0000 C CNN
+	1    6200 5000
 	1    0    0    -1
 $EndComp
@@
 P 6200 5200
 F 0 "BT1" H 6300 5300 50  0000 L CNN
-F 1 "3.7V" H 6300 5200 50  0000 L CNN
+F 1 "CR2032" H 6300 5200 50  0000 L CNN
 F 2 "Battery_Holders:Keystone_106_1x20mm-CoinCell" V 6200 5260 50  0001 C CNN
 F 3 "" V 6200 5260 50  0000 C CNN
@@
 $EndComp
 $Comp
-L GND #PWR04
+L GND #PWR22
 U 1 1 59102F4B
 P 6200 5300
-F 0 "#PWR04" H 6200 5050 50  0001 C CNN
+F 0 "#PWR22" H 6200 5050 50  0001 C CNN
 F 1 "GND" H 6200 5150 50  0000 C CNN
 F 2 "" H 6200 5300 50  0000 C CNN
@@
 ANT
 $Comp
-L GND #PWR05
+L GND #PWR30
 U 1 1 591034EC
 P 9250 3450
-F 0 "#PWR05" H 9250 3200 50  0001 C CNN
+F 0 "#PWR30" H 9250 3200 50  0001 C CNN
 F 1 "GND" H 9250 3300 50  0000 C CNN
 F 2 "" H 9250 3450 50  0000 C CNN
@@
 $EndComp
 $Comp
-L +3V3 #PWR06
+L +3V3 #PWR31
 U 1 1 59103508
 P 9250 3650
-F 0 "#PWR06" H 9250 3500 50  0001 C CNN
+F 0 "#PWR31" H 9250 3500 50  0001 C CNN
 F 1 "+3V3" H 9250 3790 50  0000 C CNN
 F 2 "" H 9250 3650 50  0000 C CNN
@@
 	1550 3850 2000 3850
 $Comp
-L GND #PWR07
+L GND #PWR2
 U 1 1 59103D18
 P 1550 3350
-F 0 "#PWR07" H 1550 3100 50  0001 C CNN
+F 0 "#PWR2" H 1550 3100 50  0001 C CNN
 F 1 "GND" H 1550 3200 50  0000 C CNN
 F 2 "" H 1550 3350 50  0000 C CNN
@@
 $EndComp
 $Comp
-L GND #PWR08
+L GND #PWR3
 U 1 1 59103D4F
 P 1550 3550
-F 0 "#PWR08" H 1550 3300 50  0001 C CNN
+F 0 "#PWR3" H 1550 3300 50  0001 C CNN
 F 1 "GND" H 1550 3400 50  0000 C CNN
 F 2 "" H 1550 3550 50  0000 C CNN
@@
 $EndComp
 $Comp
-L GND #PWR09
+L GND #PWR4
 U 1 1 59103D6D
 P 1550 3750
-F 0 "#PWR09" H 1550 3500 50  0001 C CNN
+F 0 "#PWR4" H 1550 3500 50  0001 C CNN
 F 1 "GND" H 1550 3600 50  0000 C CNN
 F 2 "" H 1550 3750 50  0000 C CNN
@@
 $EndComp
 $Comp
-L GND #PWR010
+L GND #PWR5
 U 1 1 59103DA4
 P 1550 3950
-F 0 "#PWR010" H 1550 3700 50  0001 C CNN
+F 0 "#PWR5" H 1550 3700 50  0001 C CNN
 F 1 "GND" H 1550 3800 50  0000 C CNN
 F 2 "" H 1550 3950 50  0000 C CNN
@@
 IN0
 $Comp
-L GND #PWR011
+L GND #PWR9
 U 1 1 5910458F
 P 2550 3900
-F 0 "#PWR011" H 2550 3650 50  0001 C CNN
+F 0 "#PWR9" H 2550 3650 50  0001 C CNN
 F 1 "GND" H 2550 3750 50  0000 C CNN
 F 2 "" H 2550 3900 50  0000 C CNN
@@
 $EndComp
 $Comp
-L +3V3 #PWR012
+L +3V3 #PWR8
 U 1 1 591045FE
 P 2550 3200
-F 0 "#PWR012" H 2550 3050 50  0001 C CNN
+F 0 "#PWR8" H 2550 3050 50  0001 C CNN
 F 1 "+3V3" H 2550 3340 50  0000 C CNN
 F 2 "" H 2550 3200 50  0000 C CNN
@@
 $EndComp
 $Comp
-L +3V3 #PWR013
+L +3V3 #PWR23
 U 1 1 5910481E
 P 6700 5000
-F 0 "#PWR013" H 6700 4850 50  0001 C CNN
+F 0 "#PWR23" H 6700 4850 50  0001 C CNN
 F 1 "+3V3" H 6700 5140 50  0000 C CNN
 F 2 "" H 6700 5000 50  0000 C CNN
@@
 $EndComp
 $Comp
-L GND #PWR014
+L GND #PWR24
 U 1 1 59104863
 P 6700 5300
-F 0 "#PWR014" H 6700 5050 50  0001 C CNN
+F 0 "#PWR24" H 6700 5050 50  0001 C CNN
 F 1 "GND" H 6700 5150 50  0000 C CNN
 F 2 "" H 6700 5300 50  0000 C CNN
@@
 IN1
 $Comp
-L GND #PWR015
+L GND #PWR12
 U 1 1 59104EB6
 P 3150 3900
-F 0 "#PWR015" H 3150 3650 50  0001 C CNN
+F 0 "#PWR12" H 3150 3650 50  0001 C CNN
 F 1 "GND" H 3150 3750 50  0000 C CNN
 F 2 "" H 3150 3900 50  0000 C CNN
@@
 $EndComp
 $Comp
-L +3V3 #PWR016
+L +3V3 #PWR11
 U 1 1 59104EBC
 P 3150 3200
-F 0 "#PWR016" H 3150 3050 50  0001 C CNN
+F 0 "#PWR11" H 3150 3050 50  0001 C CNN
 F 1 "+3V3" H 3150 3340 50  0000 C CNN
 F 2 "" H 3150 3200 50  0000 C CNN
@@
 IN2
 $Comp
-L GND #PWR017
+L GND #PWR14
 U 1 1 5910502C
 P 3750 3900
-F 0 "#PWR017" H 3750 3650 50  0001 C CNN
+F 0 "#PWR14" H 3750 3650 50  0001 C CNN
 F 1 "GND" H 3750 3750 50  0000 C CNN
 F 2 "" H 3750 3900 50  0000 C CNN
@@
 $EndComp
 $Comp
-L +3V3 #PWR018
+L +3V3 #PWR13
 U 1 1 59105032
 P 3750 3200
-F 0 "#PWR018" H 3750 3050 50  0001 C CNN
+F 0 "#PWR13" H 3750 3050 50  0001 C CNN
 F 1 "+3V3" H 3750 3340 50  0000 C CNN
 F 2 "" H 3750 3200 50  0000 C CNN
@@
 IN3
 $Comp
-L GND #PWR019
+L GND #PWR16
 U 1 1 59105048
 P 4350 3900
-F 0 "#PWR019" H 4350 3650 50  0001 C CNN
+F 0 "#PWR16" H 4350 3650 50  0001 C CNN
 F 1 "GND" H 4350 3750 50  0000 C CNN
 F 2 "" H 4350 3900 50  0000 C CNN
@@
 $EndComp
 $Comp
-L +3V3 #PWR020
+L +3V3 #PWR15
 U 1 1 5910504E
 P 4350 3200
-F 0 "#PWR020" H 4350 3050 50  0001 C CNN
+F 0 "#PWR15" H 4350 3050 50  0001 C CNN
 F 1 "+3V3" H 4350 3340 50  0000 C CNN
 F 2 "" H 4350 3200 50  0000 C CNN
@@
 	8250 3550 7950 3550
 $Comp
-L GND #PWR021
+L GND #PWR29
 U 1 1 59106156
 P 8800 3900
-F 0 "#PWR021" H 8800 3650 50  0001 C CNN
+F 0 "#PWR29" H 8800 3650 50  0001 C CNN
 F 1 "GND" H 8800 3750 50  0000 C CNN
 F 2 "" H 8800 3900 50  0000 C CNN
@@
 $EndComp
 $Comp
-L +3V3 #PWR022
+L +3V3 #PWR25
 U 1 1 5910891F
 P 7250 5000
-F 0 "#PWR022" H 7250 4850 50  0001 C CNN
+F 0 "#PWR25" H 7250 4850 50  0001 C CNN
 F 1 "+3V3" H 7250 5140 50  0000 C CNN
 F 2 "" H 7250 5000 50  0000 C CNN
@@
 $EndComp
 $Comp
-L GND #PWR023
+L GND #PWR26
 U 1 1 59108925
 P 7250 5300
-F 0 "#PWR023" H 7250 5050 50  0001 C CNN
+F 0 "#PWR26" H 7250 5050 50  0001 C CNN
 F 1 "GND" H 7250 5150 50  0000 C CNN
 F 2 "" H 7250 5300 50  0000 C CNN
@@
 $EndComp
 $Comp
-L +3V3 #PWR024
+L +3V3 #PWR17
 U 1 1 591067BD
 P 4350 4500
-F 0 "#PWR024" H 4350 4350 50  0001 C CNN
+F 0 "#PWR17" H 4350 4350 50  0001 C CNN
 F 1 "+3V3" H 4350 4640 50  0000 C CNN
 F 2 "" H 4350 4500 50  0000 C CNN
@@
 Connection ~ 4350 4950
 $Comp
-L GND #PWR025
+L GND #PWR18
 U 1 1 59106977
 P 4350 5500
-F 0 "#PWR025" H 4350 5250 50  0001 C CNN
+F 0 "#PWR18" H 4350 5250 50  0001 C CNN
 F 1 "GND" H 4350 5350 50  0000 C CNN
 F 2 "" H 4350 5500 50  0000 C CNN
@@
 $EndComp
 $Comp
-L GND #PWR026
+L GND #PWR7
 U 1 1 59119C8B
 P 2250 4800
-F 0 "#PWR026" H 2250 4550 50  0001 C CNN
+F 0 "#PWR7" H 2250 4550 50  0001 C CNN
 F 1 "GND" H 2250 4650 50  0000 C CNN
 F 2 "" H 2250 4800 50  0000 C CNN
@@
 $EndComp
 $Comp
-L GND #PWR027
+L GND #PWR10
 U 1 1 59119D27
 P 2800 4800
-F 0 "#PWR027" H 2800 4550 50  0001 C CNN
+F 0 "#PWR10" H 2800 4550 50  0001 C CNN
 F 1 "GND" H 2800 4650 50  0000 C CNN
 F 2 "" H 2800 4800 50  0000 C CNN
@@
 $EndComp
 $Comp
-L GND #PWR028
+L GND #PWR1
 U 1 1 59119EC9
 P 1150 4800
-F 0 "#PWR028" H 1150 4550 50  0001 C CNN
+F 0 "#PWR1" H 1150 4550 50  0001 C CNN
 F 1 "GND" H 1150 4650 50  0000 C CNN
 F 2 "" H 1150 4800 50  0000 C CNN
@@
 $EndComp
 $Comp
-L GND #PWR029
+L GND #PWR6
 U 1 1 59119ED5
 P 1700 4800
-F 0 "#PWR029" H 1700 4550 50  0001 C CNN
+F 0 "#PWR6" H 1700 4550 50  0001 C CNN
 F 1 "GND" H 1700 4650 50  0000 C CNN
 F 2 "" H 1700 4800 50  0000 C CNN
@@
 	1    0    0    -1
 $EndComp
+$Comp
+L CONN_01X01 P7
+U 1 1 5911EAC4
+P 5550 5300
+F 0 "P7" H 5550 5400 50  0000 C CNN
+F 1 "BAT+" V 5650 5300 50  0000 C CNN
+F 2 "Pin_Headers:Pin_Header_Straight_1x01" H 5550 5300 50  0001 C CNN
+F 3 "" H 5550 5300 50  0000 C CNN
+	1    5550 5300
+	0    1    1    0
+$EndComp
+$Comp
+L +3V3 #PWR19
+U 1 1 5911EF06
+P 5550 4800
+F 0 "#PWR19" H 5550 4650 50  0001 C CNN
+F 1 "+3V3" H 5550 4940 50  0000 C CNN
+F 2 "" H 5550 4800 50  0000 C CNN
+F 3 "" H 5550 4800 50  0000 C CNN
+	1    5550 4800
+	1    0    0    -1
+$EndComp
+$Comp
+L CONN_01X01 P8
+U 1 1 5912165E
+P 5550 5600
+F 0 "P8" H 5550 5700 50  0000 C CNN
+F 1 "BAT-" V 5650 5600 50  0000 C CNN
+F 2 "Pin_Headers:Pin_Header_Straight_1x01" H 5550 5600 50  0001 C CNN
+F 3 "" H 5550 5600 50  0000 C CNN
+	1    5550 5600
+	0    -1   -1   0
+$EndComp
+$Comp
+L GND #PWR20
+U 1 1 591217AB
+P 5550 5800
+F 0 "#PWR20" H 5550 5550 50  0001 C CNN
+F 1 "GND" H 5550 5650 50  0000 C CNN
+F 2 "" H 5550 5800 50  0000 C CNN
+F 3 "" H 5550 5800 50  0000 C CNN
+	1    5550 5800
+	1    0    0    -1
+$EndComp
