File: circuit2/lpcounter.kicad_pcb (KiCad board)
At the start: 2 copper layers, 85 x 54 mm, 28 parts, among them IC1 ATTINY85V-P, M1 SYN115, P1 CONN_01X08, P10 BAT-, P2 CONN_02X01, P3 Hole_3.5mm, P4 Hole_3.5mm, P5 Hole_3.5mm, P6 Hole_3.5mm, P7 BAT+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

Commit message: small PCB optimizations, moving screw connector away from CR2032 battery add top zone layer and capacitor on top
Parts:
- added C7: 100nF, Capacitors_SMD:C_1206_HandSoldering, B.Cu at (48.3, 152.5)
- C5: moved to F.Cu
- D1: footprint Diodes_SMD:MELF_Handsoldering -> Diodes_SMD:MiniMELF_Handsoldering
- moved P6 7.57 mm to (76.0, 167.5)
- moved C1 2.02 mm to (86.4, 160.8)
- moved C2 2.02 mm to (94.0, 160.8)
- moved C3 2.02 mm to (101.6, 160.8)
- moved C4 2.02 mm to (109.2, 160.8)
- moved P1 2.02 mm to (78.7, 153.2)
- moved R1 2.02 mm to (82.5, 160.8)
- moved R2 2.02 mm to (90.2, 160.8)
- moved R3 2.02 mm to (97.8, 160.8)
- moved R4 2.02 mm to (105.4, 160.8)
Routing:
- net +3V3: track 143.8 -> 158.0 mm, vias 0 -> 1
- net GND: track 41.0 -> 49.7 mm, vias 0 -> 1
- net /IN3: track 69.2 -> 72.1 mm
- net /VBAT: track 46.5 -> 48.2 mm
- net /IN1: track 40.9 -> 42.6 mm
- net /IN2: track 50.3 -> 51.8 mm
- added copper zone on F.Cu, net GND
Other:
- net class Default: via_dia 0.6 -> 1; via_drill 0.4 -> 0.5
- net class Power: via_dia 0.6 -> 1; via_drill 0.4 -> 0.5
