File: circuit2/lpcounter.sch (KiCad schematic (older format))
At the start: 26 parts, among them IC1 ATTINY85V-P, M1 SYN115, P1 CONN_01X08, P2 CONN_02X01, P3 Hole_3.5mm, P4 Hole_3.5mm, P5 Hole_3.5mm, P6 Hole_3.5mm, P7 BAT+, P8 BAT-

Commit message: optimizing PCB
Connections:
- net labels added: VBAT
- wire segments 32 -> 34
Other:
- moved on the sheet: D1
Changed lines of the file:
@@
 L D_ALT D1
 U 1 1 59102ADE
-P 5550 4950
-F 0 "D1" H 5550 5050 50  0000 C CNN
-F 1 "1N4148" H 5550 4850 50  0000 C CNN
-F 2 "Diodes_SMD:MELF_Handsoldering" H 5550 4950 50  0001 C CNN
-F 3 "" H 5550 4950 50  0000 C CNN
-	1    5550 4950
+P 5550 4700
+F 0 "D1" H 5550 4800 50  0000 C CNN
+F 1 "1N4148" H 5550 4600 50  0000 C CNN
+F 2 "Diodes_SMD:MELF_Handsoldering" H 5550 4700 50  0001 C CNN
+F 3 "" H 5550 4700 50  0000 C CNN
+	1    5550 4700
 	0    1    1    0
 $EndComp
@@
 $EndComp
 $Comp
-L GND #PWR029
-U 1 1 59119ED5
-P 1700 4800
-F 0 "#PWR029" H 1700 4550 50  0001 C CNN
-F 1 "GND" H 1700 4650 50  0000 C CNN
-F 2 "" H 1700 4800 50  0000 C CNN
-F 3 "" H 1700 4800 50  0000 C CNN
-	1    1700 4800
-	1    0    0    -1
-$EndComp
-$Comp
 L CONN_01X01 P7
 U 1 1 5911EAC4
@@
 $EndComp
 $Comp
-L +3V3 #PWR030
+L +3V3 #PWR029
 U 1 1 5911EF06
-P 5550 4800
-F 0 "#PWR030" H 5550 4650 50  0001 C CNN
-F 1 "+3V3" H 5550 4940 50  0000 C CNN
-F 2 "" H 5550 4800 50  0000 C CNN
-F 3 "" H 5550 4800 50  0000 C CNN
-	1    5550 4800
+P 5550 4550
+F 0 "#PWR029" H 5550 4400 50  0001 C CNN
+F 1 "+3V3" H 5550 4690 50  0000 C CNN
+F 2 "" H 5550 4550 50  0000 C CNN
+F 3 "" H 5550 4550 50  0000 C CNN
+	1    5550 4550
 	1    0    0    -1
 $EndComp
@@
 $EndComp
 $Comp
-L GND #PWR031
+L GND #PWR030
 U 1 1 591217AB
 P 5550 5800
-F 0 "#PWR031" H 5550 5550 50  0001 C CNN
+F 0 "#PWR030" H 5550 5550 50  0001 C CNN
 F 1 "GND" H 5550 5650 50  0000 C CNN
 F 2 "" H 5550 5800 50  0000 C CNN
@@
 Connection ~ 8800 3550
 $Comp
-L GND #PWR032
+L GND #PWR031
 U 1 1 5912DAF3
 P 9150 3900
-F 0 "#PWR032" H 9150 3650 50  0001 C CNN
+F 0 "#PWR031" H 9150 3650 50  0001 C CNN
 F 1 "GND" H 9150 3750 50  0000 C CNN
 F 2 "" H 9150 3900 50  0000 C CNN
@@
 	1    0    0    -1
 $EndComp
+Wire Wire Line
+	5550 4850 5550 5100
+Text Label 5550 5000 0    60   ~ 0
+VBAT
+Wire Wire Line
+	1700 4800 1700 4950
+Text Label 1700 4900 0    60   ~ 0
+VBAT
 $EndSCHEMATC

Commit message: changing pushbutton to jumper
Parts:
- P2: footprint Buttons_Switches_SMD:SW_SPST_SKQG -> Pin_Headers:Pin_Header_Straight_1x02
Changed lines of the file:
@@
 F 0 "P2" H 4350 5350 50  0000 C CNN
 F 1 "CONN_02X01" H 4350 5150 50  0000 C CNN
-F 2 "Buttons_Switches_SMD:SW_SPST_SKQG" H 4350 4050 50  0001 C CNN
+F 2 "Pin_Headers:Pin_Header_Straight_1x02" H 4350 4050 50  0001 C CNN
 F 3 "" H 4350 4050 50  0000 C CNN
 	1    4350 5250

Commit message: increase PCB to fully fit into ABC box, multiple battery contacts
Parts:
- added P10: BAT-, Pin_Headers:Pin_Header_Straight_1x01, symbol CONN_01X01
- added P9: BAT+, Pin_Headers:Pin_Header_Straight_1x01, symbol CONN_01X01
- C5: footprint Capacitors_Tantalum_SMD:Tantalum_Case-R_EIA-2012-12_Hand -> Capacitors_Tantalum_SMD:Tantalum_Case-U_EIA-6032-15_Hand
Connections:
- wire segments 34 -> 36
Changed lines of the file:
@@
 IN0
 $Comp
-L GND #PWR01
+L GND #PWR28
 U 1 1 591028B9
 P 7900 3850
-F 0 "#PWR01" H 7900 3600 50  0001 C CNN
+F 0 "#PWR28" H 7900 3600 50  0001 C CNN
 F 1 "GND" H 7900 3700 50  0000 C CNN
 F 2 "" H 7900 3850 50  0000 C CNN
@@
 RESETn
 $Comp
-L +3V3 #PWR02
+L +3V3 #PWR27
 U 1 1 59102AB8
 P 7900 3250
-F 0 "#PWR02" H 7900 3100 50  0001 C CNN
+F 0 "#PWR27" H 7900 3100 50  0001 C CNN
 F 1 "+3V3" H 7900 3390 50  0000 C CNN
 F 2 "" H 7900 3250 50  0000 C CNN
@@
 $EndComp
 $Comp
-L +3V3 #PWR03
+L +3V3 #PWR21
 U 1 1 59102B87
 P 6200 5000
-F 0 "#PWR03" H 6200 4850 50  0001 C CNN
+F 0 "#PWR21" H 6200 4850 50  0001 C CNN
 F 1 "+3V3" H 6200 5140 50  0000 C CNN
 F 2 "" H 6200 5000 50  0000 C CNN
@@
 $EndComp
 $Comp
-L GND #PWR04
+L GND #PWR22
 U 1 1 59102F4B
 P 6200 5300
-F 0 "#PWR04" H 6200 5050 50  0001 C CNN
+F 0 "#PWR22" H 6200 5050 50  0001 C CNN
 F 1 "GND" H 6200 5150 50  0000 C CNN
 F 2 "" H 6200 5300 50  0000 C CNN
@@
 ANT
 $Comp
-L GND #PWR05
+L GND #PWR31
 U 1 1 591034EC
 P 9750 3450
-F 0 "#PWR05" H 9750 3200 50  0001 C CNN
+F 0 "#PWR31" H 9750 3200 50  0001 C CNN
 F 1 "GND" H 9750 3300 50  0000 C CNN
 F 2 "" H 9750 3450 50  0000 C CNN
@@
 $EndComp
 $Comp
-L +3V3 #PWR06
+L +3V3 #PWR32
 U 1 1 59103508
 P 9750 3650
-F 0 "#PWR06" H 9750 3500 50  0001 C CNN
+F 0 "#PWR32" H 9750 3500 50  0001 C CNN
 F 1 "+3V3" H 9750 3790 50  0000 C CNN
 F 2 "" H 9750 3650 50  0000 C CNN
@@
 	1550 3850 2000 3850
 $Comp
-L GND #PWR07
+L GND #PWR2
 U 1 1 59103D18
 P 1550 3350
-F 0 "#PWR07" H 1550 3100 50  0001 C CNN
+F 0 "#PWR2" H 1550 3100 50  0001 C CNN
 F 1 "GND" H 1550 3200 50  0000 C CNN
 F 2 "" H 1550 3350 50  0000 C CNN
@@
 $EndComp
 $Comp
-L GND #PWR08
+L GND #PWR3
 U 1 1 59103D4F
 P 1550 3550
-F 0 "#PWR08" H 1550 3300 50  0001 C CNN
+F 0 "#PWR3" H 1550 3300 50  0001 C CNN
 F 1 "GND" H 1550 3400 50  0000 C CNN
 F 2 "" H 1550 3550 50  0000 C CNN
@@
 $EndComp
 $Comp
-L GND #PWR09
+L GND #PWR4
 U 1 1 59103D6D
 P 1550 3750
-F 0 "#PWR09" H 1550 3500 50  0001 C CNN
+F 0 "#PWR4" H 1550 3500 50  0001 C CNN
 F 1 "GND" H 1550 3600 50  0000 C CNN
 F 2 "" H 1550 3750 50  0000 C CNN
@@
 $EndComp
 $Comp
-L GND #PWR010
+L GND #PWR5
 U 1 1 59103DA4
 P 1550 3950
-F 0 "#PWR010" H 1550 3700 50  0001 C CNN
+F 0 "#PWR5" H 1550 3700 50  0001 C CNN
 F 1 "GND" H 1550 3800 50  0000 C CNN
 F 2 "" H 1550 3950 50  0000 C CNN
@@
 IN0
 $Comp
-L GND #PWR011
+L GND #PWR8
 U 1 1 5910458F
 P 2550 3900
-F 0 "#PWR011" H 2550 3650 50  0001 C CNN
+F 0 "#PWR8" H 2550 3650 50  0001 C CNN
 F 1 "GND" H 2550 3750 50  0000 C CNN
 F 2 "" H 2550 3900 50  0000 C CNN
@@
 $EndComp
 $Comp
-L +3V3 #PWR012
+L +3V3 #PWR7
 U 1 1 591045FE
 P 2550 3200
-F 0 "#PWR012" H 2550 3050 50  0001 C CNN
+F 0 "#PWR7" H 2550 3050 50  0001 C CNN
 F 1 "+3V3" H 2550 3340 50  0000 C CNN
 F 2 "" H 2550 3200 50  0000 C CNN
@@
 $EndComp
 $Comp
-L +3V3 #PWR013
+L +3V3 #PWR23
 U 1 1 5910481E
 P 6700 5000
-F 0 "#PWR013" H 6700 4850 50  0001 C CNN
+F 0 "#PWR23" H 6700 4850 50  0001 C CNN
 F 1 "+3V3" H 6700 5140 50  0000 C CNN
 F 2 "" H 6700 5000 50  0000 C CNN
@@
 $EndComp
 $Comp
-L GND #PWR014
+L GND #PWR24
 U 1 1 59104863
 P 6700 5300
-F 0 "#PWR014" H 6700 5050 50  0001 C CNN
+F 0 "#PWR24" H 6700 5050 50  0001 C CNN
 F 1 "GND" H 6700 5150 50  0000 C CNN
 F 2 "" H 6700 5300 50  0000 C CNN
@@
 F 0 "C5" H 6725 5250 50  0000 L CNN
 F 1 "4.7uF" H 6725 5050 50  0000 L CNN
-F 2 "Capacitors_Tantalum_SMD:Tantalum_Case-R_EIA-2012-12_Hand" H 6738 5000 50  0001 C CNN
+F 2 "Capacitors_Tantalum_SMD:Tantalum_Case-U_EIA-6032-15_Hand" H 6738 5000 50  0001 C CNN
 F 3 "" H 6700 5150 50  0000 C CNN
 	1    6700 5150
@@
 IN1
 $Comp
-L GND #PWR015
+L GND #PWR11
 U 1 1 59104EB6
 P 3150 3900
-F 0 "#PWR015" H 3150 3650 50  0001 C CNN
+F 0 "#PWR11" H 3150 3650 50  0001 C CNN
 F 1 "GND" H 3150 3750 50  0000 C CNN
 F 2 "" H 3150 3900 50  0000 C CNN
@@
 $EndComp
 $Comp
-L +3V3 #PWR016
+L +3V3 #PWR10
 U 1 1 59104EBC
 P 3150 3200
-F 0 "#PWR016" H 3150 3050 50  0001 C CNN
+F 0 "#PWR10" H 3150 3050 50  0001 C CNN
 F 1 "+3V3" H 3150 3340 50  0000 C CNN
 F 2 "" H 3150 3200 50  0000 C CNN
@@
 IN2
 $Comp
-L GND #PWR017
+L GND #PWR13
 U 1 1 5910502C
 P 3750 3900
-F 0 "#PWR017" H 3750 3650 50  0001 C CNN
+F 0 "#PWR13" H 3750 3650 50  0001 C CNN
 F 1 "GND" H 3750 3750 50  0000 C CNN
 F 2 "" H 3750 3900 50  0000 C CNN
@@
 $EndComp
 $Comp
-L +3V3 #PWR018
+L +3V3 #PWR12
 U 1 1 59105032
 P 3750 3200
-F 0 "#PWR018" H 3750 3050 50  0001 C CNN
+F 0 "#PWR12" H 3750 3050 50  0001 C CNN
 F 1 "+3V3" H 3750 3340 50  0000 C CNN
 F 2 "" H 3750 3200 50  0000 C CNN
@@
 IN3
 $Comp
-L GND #PWR019
+L GND #PWR15
 U 1 1 59105048
 P 4350 3900
-F 0 "#PWR019" H 4350 3650 50  0001 C CNN
+F 0 "#PWR15" H 4350 3650 50  0001 C CNN
 F 1 "GND" H 4350 3750 50  0000 C CNN
 F 2 "" H 4350 3900 50  0000 C CNN
@@
 $EndComp
 $Comp
-L +3V3 #PWR020
+L +3V3 #PWR14
 U 1 1 5910504E
 P 4350 3200
-F 0 "#PWR020" H 4350 3050 50  0001 C CNN
+F 0 "#PWR14" H 4350 3050 50  0001 C CNN
 F 1 "+3V3" H 4350 3340 50  0000 C CNN
 F 2 "" H 4350 3200 50  0000 C CNN
@@
 	8250 3550 7950 3550
 $Comp
-L GND #PWR021
+L GND #PWR29
 U 1 1 59106156
 P 8800 3900
-F 0 "#PWR021" H 8800 3650 50  0001 C CNN
+F 0 "#PWR29" H 8800 3650 50  0001 C CNN
 F 1 "GND" H 8800 3750 50  0000 C CNN
 F 2 "" H 8800 3900 50  0000 C CNN
@@
 $EndComp
 $Comp
-L +3V3 #PWR022
+L +3V3 #PWR25
 U 1 1 5910891F
 P 7250 5000
-F 0 "#PWR022" H 7250 4850 50  0001 C CNN
+F 0 "#PWR25" H 7250 4850 50  0001 C CNN
 F 1 "+3V3" H 7250 5140 50  0000 C CNN
 F 2 "" H 7250 5000 50  0000 C CNN
@@
 $EndComp
 $Comp
-L GND #PWR023
+L GND #PWR26
 U 1 1 59108925
 P 7250 5300
-F 0 "#PWR023" H 7250 5050 50  0001 C CNN
+F 0 "#PWR26" H 7250 5050 50  0001 C CNN
 F 1 "GND" H 7250 5150 50  0000 C CNN
 F 2 "" H 7250 5300 50  0000 C CNN
@@
 $EndComp
 $Comp
-L +3V3 #PWR024
+L +3V3 #PWR16
 U 1 1 591067BD
 P 4350 4500
-F 0 "#PWR024" H 4350 4350 50  0001 C CNN
+F 0 "#PWR16" H 4350 4350 50  0001 C CNN
 F 1 "+3V3" H 4350 4640 50  0000 C CNN
 F 2 "" H 4350 4500 50  0000 C CNN
@@
 Connection ~ 4350 4950
 $Comp
-L GND #PWR025
+L GND #PWR17
 U 1 1 59106977
 P 4350 5500
-F 0 "#PWR025" H 4350 5250 50  0001 C CNN
+F 0 "#PWR17" H 4350 5250 50  0001 C CNN
 F 1 "GND" H 4350 5350 50  0000 C CNN
 F 2 "" H 4350 5500 50  0000 C CNN
@@
 $EndComp
 $Comp
-L GND #PWR026
+L GND #PWR6
 U 1 1 59119C8B
 P 2250 4800
-F 0 "#PWR026" H 2250 4550 50  0001 C CNN
+F 0 "#PWR6" H 2250 4550 50  0001 C CNN
 F 1 "GND" H 2250 4650 50  0000 C CNN
 F 2 "" H 2250 4800 50  0000 C CNN
@@
 $EndComp
 $Comp
-L GND #PWR027
+L GND #PWR9
 U 1 1 59119D27
 P 2800 4800
-F 0 "#PWR027" H 2800 4550 50  0001 C CNN
+F 0 "#PWR9" H 2800 4550 50  0001 C CNN
 F 1 "GND" H 2800 4650 50  0000 C CNN
 F 2 "" H 2800 4800 50  0000 C CNN
@@
 $EndComp
 $Comp
-L GND #PWR028
+L GND #PWR1
 U 1 1 59119EC9
 P 1150 4800
-F 0 "#PWR028" H 1150 4550 50  0001 C CNN
+F 0 "#PWR1" H 1150 4550 50  0001 C CNN
 F 1 "GND" H 1150 4650 50  0000 C CNN
 F 2 "" H 1150 4800 50  0000 C CNN
@@
 $EndComp
 $Comp
-L +3V3 #PWR029
+L +3V3 #PWR19
 U 1 1 5911EF06
 P 5550 4550
-F 0 "#PWR029" H 5550 4400 50  0001 C CNN
+F 0 "#PWR19" H 5550 4400 50  0001 C CNN
 F 1 "+3V3" H 5550 4690 50  0000 C CNN
 F 2 "" H 5550 4550 50  0000 C CNN
@@
 $EndComp
 $Comp
-L GND #PWR030
+L GND #PWR20
 U 1 1 591217AB
 P 5550 5800
-F 0 "#PWR030" H 5550 5550 50  0001 C CNN
+F 0 "#PWR20" H 5550 5550 50  0001 C CNN
 F 1 "GND" H 5550 5650 50  0000 C CNN
 F 2 "" H 5550 5800 50  0000 C CNN
@@
 Connection ~ 8800 3550
 $Comp
-L GND #PWR031
+L GND #PWR30
 U 1 1 5912DAF3
 P 9150 3900
-F 0 "#PWR031" H 9150 3650 50  0001 C CNN
+F 0 "#PWR30" H 9150 3650 50  0001 C CNN
 F 1 "GND" H 9150 3750 50  0000 C CNN
 F 2 "" H 9150 3900 50  0000 C CNN
@@
 Text Label 1700 4900 0    60   ~ 0
 VBAT
+$Comp
+L CONN_01X01 P9
+U 1 1 5917212A
+P 5250 5300
+F 0 "P9" H 5250 5400 50  0000 C CNN
+F 1 "BAT+" V 5350 5300 50  0000 C CNN
+F 2 "Pin_Headers:Pin_Header_Straight_1x01" H 5250 5300 50  0001 C CNN
+F 3 "" H 5250 5300 50  0000 C CNN
+	1    5250 5300
+	0    1    1    0
+$EndComp
+$Comp
+L CONN_01X01 P10
+U 1 1 5917221C
+P 5250 5600
+F 0 "P10" H 5250 5700 50  0000 C CNN
+F 1 "BAT-" V 5350 5600 50  0000 C CNN
+F 2 "Pin_Headers:Pin_Header_Straight_1x01" H 5250 5600 50  0001 C CNN
+F 3 "" H 5250 5600 50  0000 C CNN
+	1    5250 5600
+	0    -1   -1   0
+$EndComp
+$Comp
+L GND #PWR18
+U 1 1 59172348
+P 5250 5800
+F 0 "#PWR18" H 5250 5550 50  0001 C CNN
+F 1 "GND" H 5250 5650 50  0000 C CNN
+F 2 "" H 5250 5800 50  0000 C CNN
+F 3 "" H 5250 5800 50  0000 C CNN
+	1    5250 5800
+	1    0    0    -1
+$EndComp
+Wire Wire Line
+	5250 5100 5250 5000
+Wire Wire Line
+	5250 5000 5550 5000
+Connection ~ 5550 5000
 $EndSCHEMATC

Commit message: holes update
Parts:
- P3, P4, P5, P6: footprint Mounting_Holes:MountingHole_3.5mm -> Mounting_Holes:MountingHole_3.5mm_Pad
Changed lines of the file:
@@
 IN0
 $Comp
-L GND #PWR28
+L GND #PWR01
 U 1 1 591028B9
 P 7900 3850
-F 0 "#PWR28" H 7900 3600 50  0001 C CNN
+F 0 "#PWR01" H 7900 3600 50  0001 C CNN
 F 1 "GND" H 7900 3700 50  0000 C CNN
 F 2 "" H 7900 3850 50  0000 C CNN
@@
 RESETn
 $Comp
-L +3V3 #PWR27
+L +3V3 #PWR02
 U 1 1 59102AB8
 P 7900 3250
-F 0 "#PWR27" H 7900 3100 50  0001 C CNN
+F 0 "#PWR02" H 7900 3100 50  0001 C CNN
 F 1 "+3V3" H 7900 3390 50  0000 C CNN
 F 2 "" H 7900 3250 50  0000 C CNN
@@
 $EndComp
 $Comp
-L +3V3 #PWR21
+L +3V3 #PWR03
 U 1 1 59102B87
 P 6200 5000
-F 0 "#PWR21" H 6200 4850 50  0001 C CNN
+F 0 "#PWR03" H 6200 4850 50  0001 C CNN
 F 1 "+3V3" H 6200 5140 50  0000 C CNN
 F 2 "" H 6200 5000 50  0000 C CNN
@@
 $EndComp
 $Comp
-L GND #PWR22
+L GND #PWR04
 U 1 1 59102F4B
 P 6200 5300
-F 0 "#PWR22" H 6200 5050 50  0001 C CNN
+F 0 "#PWR04" H 6200 5050 50  0001 C CNN
 F 1 "GND" H 6200 5150 50  0000 C CNN
 F 2 "" H 6200 5300 50  0000 C CNN
@@
 ANT
 $Comp
-L GND #PWR31
+L GND #PWR05
 U 1 1 591034EC
 P 9750 3450
-F 0 "#PWR31" H 9750 3200 50  0001 C CNN
+F 0 "#PWR05" H 9750 3200 50  0001 C CNN
 F 1 "GND" H 9750 3300 50  0000 C CNN
 F 2 "" H 9750 3450 50  0000 C CNN
@@
 $EndComp
 $Comp
-L +3V3 #PWR32
+L +3V3 #PWR06
 U 1 1 59103508
 P 9750 3650
-F 0 "#PWR32" H 9750 3500 50  0001 C CNN
+F 0 "#PWR06" H 9750 3500 50  0001 C CNN
 F 1 "+3V3" H 9750 3790 50  0000 C CNN
 F 2 "" H 9750 3650 50  0000 C CNN
@@
 	1550 3850 2000 3850
 $Comp
-L GND #PWR2
+L GND #PWR07
 U 1 1 59103D18
 P 1550 3350
-F 0 "#PWR2" H 1550 3100 50  0001 C CNN
+F 0 "#PWR07" H 1550 3100 50  0001 C CNN
 F 1 "GND" H 1550 3200 50  0000 C CNN
 F 2 "" H 1550 3350 50  0000 C CNN
@@
 $EndComp
 $Comp
-L GND #PWR3
+L GND #PWR08
 U 1 1 59103D4F
 P 1550 3550
-F 0 "#PWR3" H 1550 3300 50  0001 C CNN
+F 0 "#PWR08" H 1550 3300 50  0001 C CNN
 F 1 "GND" H 1550 3400 50  0000 C CNN
 F 2 "" H 1550 3550 50  0000 C CNN
@@
 $EndComp
 $Comp
-L GND #PWR4
+L GND #PWR09
 U 1 1 59103D6D
 P 1550 3750
-F 0 "#PWR4" H 1550 3500 50  0001 C CNN
+F 0 "#PWR09" H 1550 3500 50  0001 C CNN
 F 1 "GND" H 1550 3600 50  0000 C CNN
 F 2 "" H 1550 3750 50  0000 C CNN
@@
 $EndComp
 $Comp
-L GND #PWR5
+L GND #PWR010
 U 1 1 59103DA4
 P 1550 3950
-F 0 "#PWR5" H 1550 3700 50  0001 C CNN
+F 0 "#PWR010" H 1550 3700 50  0001 C CNN
 F 1 "GND" H 1550 3800 50  0000 C CNN
 F 2 "" H 1550 3950 50  0000 C CNN
@@
 IN0
 $Comp
-L GND #PWR8
+L GND #PWR011
 U 1 1 5910458F
 P 2550 3900
-F 0 "#PWR8" H 2550 3650 50  0001 C CNN
+F 0 "#PWR011" H 2550 3650 50  0001 C CNN
 F 1 "GND" H 2550 3750 50  0000 C CNN
 F 2 "" H 2550 3900 50  0000 C CNN
@@
 $EndComp
 $Comp
-L +3V3 #PWR7
+L +3V3 #PWR012
 U 1 1 591045FE
 P 2550 3200
-F 0 "#PWR7" H 2550 3050 50  0001 C CNN
+F 0 "#PWR012" H 2550 3050 50  0001 C CNN
 F 1 "+3V3" H 2550 3340 50  0000 C CNN
 F 2 "" H 2550 3200 50  0000 C CNN
@@
 $EndComp
 $Comp
-L +3V3 #PWR23
+L +3V3 #PWR013
 U 1 1 5910481E
 P 6700 5000
-F 0 "#PWR23" H 6700 4850 50  0001 C CNN
+F 0 "#PWR013" H 6700 4850 50  0001 C CNN
 F 1 "+3V3" H 6700 5140 50  0000 C CNN
 F 2 "" H 6700 5000 50  0000 C CNN
@@
 $EndComp
 $Comp
-L GND #PWR24
+L GND #PWR014
 U 1 1 59104863
 P 6700 5300
-F 0 "#PWR24" H 6700 5050 50  0001 C CNN
+F 0 "#PWR014" H 6700 5050 50  0001 C CNN
 F 1 "GND" H 6700 5150 50  0000 C CNN
 F 2 "" H 6700 5300 50  0000 C CNN
@@
 IN1
 $Comp
-L GND #PWR11
+L GND #PWR015
 U 1 1 59104EB6
 P 3150 3900
-F 0 "#PWR11" H 3150 3650 50  0001 C CNN
+F 0 "#PWR015" H 3150 3650 50  0001 C CNN
 F 1 "GND" H 3150 3750 50  0000 C CNN
 F 2 "" H 3150 3900 50  0000 C CNN
@@
 $EndComp
 $Comp
-L +3V3 #PWR10
+L +3V3 #PWR016
 U 1 1 59104EBC
 P 3150 3200
-F 0 "#PWR10" H 3150 3050 50  0001 C CNN
+F 0 "#PWR016" H 3150 3050 50  0001 C CNN
 F 1 "+3V3" H 3150 3340 50  0000 C CNN
 F 2 "" H 3150 3200 50  0000 C CNN
@@
 IN2
 $Comp
-L GND #PWR13
+L GND #PWR017
 U 1 1 5910502C
 P 3750 3900
-F 0 "#PWR13" H 3750 3650 50  0001 C CNN
+F 0 "#PWR017" H 3750 3650 50  0001 C CNN
 F 1 "GND" H 3750 3750 50  0000 C CNN
 F 2 "" H 3750 3900 50  0000 C CNN
@@
 $EndComp
 $Comp
-L +3V3 #PWR12
+L +3V3 #PWR018
 U 1 1 59105032
 P 3750 3200
-F 0 "#PWR12" H 3750 3050 50  0001 C CNN
+F 0 "#PWR018" H 3750 3050 50  0001 C CNN
 F 1 "+3V3" H 3750 3340 50  0000 C CNN
 F 2 "" H 3750 3200 50  0000 C CNN
@@
 IN3
 $Comp
-L GND #PWR15
+L GND #PWR019
 U 1 1 59105048
 P 4350 3900
-F 0 "#PWR15" H 4350 3650 50  0001 C CNN
+F 0 "#PWR019" H 4350 3650 50  0001 C CNN
 F 1 "GND" H 4350 3750 50  0000 C CNN
 F 2 "" H 4350 3900 50  0000 C CNN
@@
 $EndComp
 $Comp
-L +3V3 #PWR14
+L +3V3 #PWR020
 U 1 1 5910504E
 P 4350 3200
-F 0 "#PWR14" H 4350 3050 50  0001 C CNN
+F 0 "#PWR020" H 4350 3050 50  0001 C CNN
 F 1 "+3V3" H 4350 3340 50  0000 C CNN
 F 2 "" H 4350 3200 50  0000 C CNN
@@
 	8250 3550 7950 3550
 $Comp
-L GND #PWR29
+L GND #PWR021
 U 1 1 59106156
 P 8800 3900
-F 0 "#PWR29" H 8800 3650 50  0001 C CNN
+F 0 "#PWR021" H 8800 3650 50  0001 C CNN
 F 1 "GND" H 8800 3750 50  0000 C CNN
 F 2 "" H 8800 3900 50  0000 C CNN
@@
 $EndComp
 $Comp
-L +3V3 #PWR25
+L +3V3 #PWR022
 U 1 1 5910891F
 P 7250 5000
-F 0 "#PWR25" H 7250 4850 50  0001 C CNN
+F 0 "#PWR022" H 7250 4850 50  0001 C CNN
 F 1 "+3V3" H 7250 5140 50  0000 C CNN
 F 2 "" H 7250 5000 50  0000 C CNN
@@
 $EndComp
 $Comp
-L GND #PWR26
+L GND #PWR023
 U 1 1 59108925
 P 7250 5300
-F 0 "#PWR26" H 7250 5050 50  0001 C CNN
+F 0 "#PWR023" H 7250 5050 50  0001 C CNN
 F 1 "GND" H 7250 5150 50  0000 C CNN
 F 2 "" H 7250 5300 50  0000 C CNN
@@
 $EndComp
 $Comp
-L +3V3 #PWR16
+L +3V3 #PWR024
 U 1 1 591067BD
 P 4350 4500
-F 0 "#PWR16" H 4350 4350 50  0001 C CNN
+F 0 "#PWR024" H 4350 4350 50  0001 C CNN
 F 1 "+3V3" H 4350 4640 50  0000 C CNN
 F 2 "" H 4350 4500 50  0000 C CNN
@@
 Connection ~ 4350 4950
 $Comp
-L GND #PWR17
+L GND #PWR025
 U 1 1 59106977
 P 4350 5500
-F 0 "#PWR17" H 4350 5250 50  0001 C CNN
+F 0 "#PWR025" H 4350 5250 50  0001 C CNN
 F 1 "GND" H 4350 5350 50  0000 C CNN
 F 2 "" H 4350 5500 50  0000 C CNN
@@
 F 0 "P5" H 2250 4700 50  0000 C CNN
 F 1 "Hole_3.5mm" V 2350 4600 50  0000 C CNN
-F 2 "Mounting_Holes:MountingHole_3.5mm" H 2250 4600 50  0001 C CNN
+F 2 "Mounting_Holes:MountingHole_3.5mm_Pad" H 2250 4600 50  0001 C CNN
 F 3 "" H 2250 4600 50  0000 C CNN
 	1    2250 4600
@@
 $EndComp
 $Comp
-L GND #PWR6
+L GND #PWR026
 U 1 1 59119C8B
 P 2250 4800
-F 0 "#PWR6" H 2250 4550 50  0001 C CNN
+F 0 "#PWR026" H 2250 4550 50  0001 C CNN
 F 1 "GND" H 2250 4650 50  0000 C CNN
 F 2 "" H 2250 4800 50  0000 C CNN
@@
 F 0 "P6" H 2800 4700 50  0000 C CNN
 F 1 "Hole_3.5mm" V 2900 4600 50  0000 C CNN
-F 2 "Mounting_Holes:MountingHole_3.5mm" H 2800 4600 50  0001 C CNN
+F 2 "Mounting_Holes:MountingHole_3.5mm_Pad" H 2800 4600 50  0001 C CNN
 F 3 "" H 2800 4600 50  0000 C CNN
 	1    2800 4600
@@
 $EndComp
 $Comp
-L GND #PWR9
+L GND #PWR027
 U 1 1 59119D27
 P 2800 4800
-F 0 "#PWR9" H 2800 4550 50  0001 C CNN
+F 0 "#PWR027" H 2800 4550 50  0001 C CNN
 F 1 "GND" H 2800 4650 50  0000 C CNN
 F 2 "" H 2800 4800 50  0000 C CNN
@@
 F 0 "P3" H 1150 4700 50  0000 C CNN
 F 1 "Hole_3.5mm" V 1250 4600 50  0000 C CNN
-F 2 "Mounting_Holes:MountingHole_3.5mm" H 1150 4600 50  0001 C CNN
+F 2 "Mounting_Holes:MountingHole_3.5mm_Pad" H 1150 4600 50  0001 C CNN
 F 3 "" H 1150 4600 50  0000 C CNN
 	1    1150 4600
@@
 $EndComp
 $Comp
-L GND #PWR1
+L GND #PWR028
 U 1 1 59119EC9
 P 1150 4800
-F 0 "#PWR1" H 1150 4550 50  0001 C CNN
+F 0 "#PWR028" H 1150 4550 50  0001 C CNN
 F 1 "GND" H 1150 4650 50  0000 C CNN
 F 2 "" H 1150 4800 50  0000 C CNN
@@
 F 0 "P4" H 1700 4700 50  0000 C CNN
 F 1 "Hole_3.5mm" V 1800 4600 50  0000 C CNN
-F 2 "Mounting_Holes:MountingHole_3.5mm" H 1700 4600 50  0001 C CNN
+F 2 "Mounting_Holes:MountingHole_3.5mm_Pad" H 1700 4600 50  0001 C CNN
 F 3 "" H 1700 4600 50  0000 C CNN
 	1    1700 4600
@@
 $EndComp
 $Comp
-L +3V3 #PWR19
+L +3V3 #PWR029
 U 1 1 5911EF06
 P 5550 4550
-F 0 "#PWR19" H 5550 4400 50  0001 C CNN
+F 0 "#PWR029" H 5550 4400 50  0001 C CNN
 F 1 "+3V3" H 5550 4690 50  0000 C CNN
 F 2 "" H 5550 4550 50  0000 C CNN
@@
 $EndComp
 $Comp
-L GND #PWR20
+L GND #PWR030
 U 1 1 591217AB
 P 5550 5800
-F 0 "#PWR20" H 5550 5550 50  0001 C CNN
+F 0 "#PWR030" H 5550 5550 50  0001 C CNN
 F 1 "GND" H 5550 5650 50  0000 C CNN
 F 2 "" H 5550 5800 50  0000 C CNN
@@
 Connection ~ 8800 3550
 $Comp
-L GND #PWR30
+L GND #PWR031
 U 1 1 5912DAF3
 P 9150 3900
-F 0 "#PWR30" H 9150 3650 50  0001 C CNN
+F 0 "#PWR031" H 9150 3650 50  0001 C CNN
 F 1 "GND" H 9150 3750 50  0000 C CNN
 F 2 "" H 9150 3900 50  0000 C CNN
@@
 $EndComp
 $Comp
-L GND #PWR18
+L GND #PWR032
 U 1 1 59172348
 P 5250 5800
-F 0 "#PWR18" H 5250 5550 50  0001 C CNN
+F 0 "#PWR032" H 5250 5550 50  0001 C CNN
 F 1 "GND" H 5250 5650 50  0000 C CNN
 F 2 "" H 5250 5800 50  0000 C CNN
